File: circuit/kicad/likepro/stm32jlc/stm32jlc.kicad_pcb (KiCad board)
At the start: 2 copper layers, 73.2 x 37.1 mm, 29 parts, among them J1 USB_B_Micro, J2 Conn_01x04_Male, J3 Conn_01x20_Male, J4 Conn_01x20_Male, SW1 SW_Push, SW2 SW_Push, U1 AMS1117-3.3, U2 STM32F103C8Tx

Commit message: KiCAD JLC
Parts:
- moved J1 0.55 mm to (175.8, 85.1)
Routing:
- net GND: track 251.8 -> 178.4 mm
- net +3.3V: track 194.3 -> 151.4 mm
- net USB_DP: track 30.1 -> 30.7 mm
- net USB_DM: track 27.6 -> 28.2 mm
- net +5V: track 8.44 -> 8.99 mm
- added copper zone on F.Cu, net +3.3V
- added copper zone on B.Cu, net GND
- removed copper zone on B.Cu, net (none)
- removed copper zone on F.Cu, net (none)

Commit message: KiCAD JLC Tutorial
Routing:
- net GND: track 178.4 -> 153.3 mm
