File: circuit/kicad/ft232_usb/ft232_usb.kicad_sch (KiCad schematic)
At the start: 19 parts, among them J1 Conn_01x03_Male, J2 Conn_01x05_Male, J3 USB_B_Micro, U1 FT232RL

Commit message: Migrate Eagle-KiCAD: FT232RL
Parts:
- C1, C2: footprint (none) -> Capacitor_SMD:C_0805_2012Metric_Pad1.18x1.45mm_HandSolder
- D1, D2, D3: footprint (none) -> LED_SMD:LED_0805_2012Metric_Pad1.15x1.40mm_HandSolder
- H1, H2, H3, H4: renamed from H?; footprint (none) -> MountingHole:MountingHole_2.2mm_M2_ISO7380_Pad
- J-HC51: footprint (none) -> Connector_PinSocket_2.54mm:PinSocket_1x06_P2.54mm_Vertical
- J1: footprint (none) -> Connector_PinHeader_2.54mm:PinHeader_1x03_P2.54mm_Vertical
- J2: footprint (none) -> Connector_PinHeader_2.54mm:PinHeader_1x05_P2.54mm_Vertical
- J3: footprint (none) -> Connector_USB:USB_Micro-B_Wuerth_629105150521
- R1, R2, R3, R4, R5: footprint (none) -> Resistor_SMD:R_0805_2012Metric_Pad1.20x1.40mm_HandSolder
Connections:
- no-connect marks 3 -> 18

Commit message: Migrate Eagle-KiCAD: USBASP
Connections:
- no-connect marks 18 -> 17
Changed lines of the file:
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@@
   (junction (at 64.77 85.09) (diameter 0) (color 0 0 0 0)
+  )
+  (junction (at 67.31 33.02) (diameter 0) (color 0 0 0 0)
   )
   (junction (at 72.39 85.09) (diameter 0) (color 0 0 0 0)
@@
   (no_connect (at 90.17 73.66))
   (no_connect (at 73.66 115.57))
-  (no_connect (at 76.2 95.25))
   (no_connect (at 90.17 76.2))
   (no_connect (at 49.53 58.42))
@@
     (stroke (width 0) (type default) (color 0 0 0 0))
   )
+  (wire (pts (xy 72.39 29.21) (xy 72.39 33.02))
+    (stroke (width 0) (type default) (color 0 0 0 0))
+  )
+  (wire (pts (xy 60.96 31.75) (xy 60.96 33.02))
+    (stroke (width 0) (type default) (color 0 0 0 0))
+  )
   (wire (pts (xy 74.93 83.82) (xy 74.93 85.09))
     (stroke (width 0) (type default) (color 0 0 0 0))
@@
     (stroke (width 0) (type default) (color 0 0 0 0))
   )
+  (wire (pts (xy 60.96 33.02) (xy 67.31 33.02))
+    (stroke (width 0) (type default) (color 0 0 0 0))
+  )
   (wire (pts (xy 69.85 85.09) (xy 64.77 85.09))
     (stroke (width 0) (type default) (color 0 0 0 0))
@@
   )
   (wire (pts (xy 97.79 66.04) (xy 109.22 66.04))
+    (stroke (width 0) (type default) (color 0 0 0 0))
+  )
+  (wire (pts (xy 67.31 31.75) (xy 67.31 33.02))
     (stroke (width 0) (type default) (color 0 0 0 0))
   )
@@
     )
   )
-  (global_label "VIO" (shape input) (at 67.31 33.02 90) (fields_autoplaced)
-    (effects (font (size 1.27 1.27)) (justify left))
-    (property "Intersheet References" "${INTERSHEET_REFS}" (id 0) (at 67.2306 27.5831 90)
+  (global_label "VIO" (shape input) (at 67.31 31.75 90) (fields_autoplaced)
+    (effects (font (size 1.27 1.27)) (justify left))
+    (property "Intersheet References" "${INTERSHEET_REFS}" (id 0) (at 67.2306 26.3131 90)
       (effects (font (size 1.27 1.27)) (justify left) hide)
     )
@@
     )
     (property "Datasheet" "" (id 3) (at 87.63 113.03 0)
+      (effects (font (size 1.27 1.27)) hide)
+    )
+    (pin "1")
+  )
+  (symbol (lib_id "power:PWR_FLAG") (at 60.96 31.75 0) (unit 1)
+    (in_bom yes) (on_board yes) (fields_autoplaced)
+    (property "Reference" "#FLG0101" (id 0) (at 60.96 29.845 0)
+      (effects (font (size 1.27 1.27)) hide)
+    )
+    (property "Value" "PWR_FLAG" (id 1) (at 60.96 26.67 0))
+    (property "Footprint" "" (id 2) (at 60.96 31.75 0)
+      (effects (font (size 1.27 1.27)) hide)
+    )
+    (property "Datasheet" "~" (id 3) (at 60.96 31.75 0)
       (effects (font (size 1.27 1.27)) hide)
     )
@@
     (pin "1")
   )
-  (symbol (lib_id "power:VCC") (at 72.39 33.02 0) (unit 1)
-    (in_bom yes) (on_board yes) (fields_autoplaced)
-    (property "Reference" "#PWR09" (id 0) (at 72.39 36.83 0)
-      (effects (font (size 1.27 1.27)) hide)
-    )
-    (property "Value" "VCC" (id 1) (at 72.39 27.94 0))
-    (property "Footprint" "" (id 2) (at 72.39 33.02 0)
-      (effects (font (size 1.27 1.27)) hide)
-    )
-    (property "Datasheet" "" (id 3) (at 72.39 33.02 0)
+  (symbol (lib_id "power:VCC") (at 72.39 29.21 0) (unit 1)
+    (in_bom yes) (on_board yes) (fields_autoplaced)
+    (property "Reference" "#PWR09" (id 0) (at 72.39 33.02 0)
+      (effects (font (size 1.27 1.27)) hide)
+    )
+    (property "Value" "VCC" (id 1) (at 72.39 24.13 0))
+    (property "Footprint" "" (id 2) (at 72.39 29.21 0)
+      (effects (font (size 1.27 1.27)) hide)
+    )
+    (property "Datasheet" "" (id 3) (at 72.39 29.21 0)
       (effects (font (size 1.27 1.27)) hide)
     )
@@
   )
   (symbol_instances
+    (path "/8bbb986c-96ec-4dd5-94c6-60285ec0fcb0"
+      (reference "#FLG0101") (unit 1) (value "PWR_FLAG") (footprint "")
+    )
     (path "/bf43e40b-9ad1-4518-a751-b0afa00edde0"
       (reference "#PWR01") (unit 1) (value "VDD") (footprint "")
