File: circuit/kicad/stm32pp/stm32pp.kicad_sch (KiCad schematic)
At the start: 33 parts, among them J1 USB_B_Micro, J2 USB_B_Micro, J3 Conn_01x04_Male, J4 Conn_01x08_Male, J5 Conn_01x08_Male, J6 Conn_01x08_Male, J7 Conn_01x08_Male, SW1 SW_Push, SW2 SW_Push, SW3 SW_Push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

Commit message: STM32PP
Parts:
- added J8: Conn_01x02_Male, symbol Connector:Conn_01x02_Male
- gave numbers to parts that had none: 4
Connections:
- net +5V: now also J8.1 (Pin_1)
- net GND: now also J8.2 (Pin_2)
Other:
- note added: "Buttons LEDs"
- note added: "Main Chip"
- note added: "Pin Header"
- note added: "USB Ports"
- note added: "Voltage Regulator"
- moved on the sheet: C1, C2, C3, C4, C5, C6, C7, C8, D1, D2, H1, H2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

Commit message: STM32PP
Parts:
- removed H1, H2, H3, H4: MountingHole, symbol Mechanical:MountingHole
- C1, C3, C4, C5, C6, C7, C8: footprint (none) -> Capacitor_SMD:C_0603_1608Metric
- C2: footprint (none) -> Capacitor_SMD:CP_Elec_3x5.3
- D1, D2: footprint (none) -> LED_SMD:LED_0805_2012Metric
- J1, J2: footprint (none) -> Connector_USB:USB_Micro-B_Wuerth_629105150521
- J3: footprint (none) -> Connector_PinHeader_2.54mm:PinHeader_1x04_P2.54mm_Vertical
- J4, J5, J6, J7: footprint (none) -> Connector_PinHeader_2.54mm:PinHeader_1x08_P2.54mm_Vertical
- J8: footprint (none) -> Connector_PinHeader_2.54mm:PinHeader_1x02_P2.54mm_Vertical
- R1, R2, R3, R4, R5, R6: footprint (none) -> Resistor_SMD:R_0603_1608Metric
- SW1, SW2, SW3: footprint (none) -> Button_Switch_SMD:SW_SPST_B3U-1000P-B
Other:
- moved on the sheet: C1, C2, C3, C4, C5, C6, C7, C8, D1, D2, J1, J2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
