File: circuit/kicad/qfp64minsys/qfp64.kicad_pcb (KiCad board)
At the start: 2 copper layers, 69.4 x 37.9 mm, 34 parts, among them J1 Conn_01x09_Pin, J10 Conn_01x03_Pin, J11 Conn_01x03_Pin, J12 Conn_01x03_Pin, J2 Conn_01x09_Pin, J3 USB_B_Mini, J4 USB_B_Mini, J5 Conn_01x03_Pin, J6 Conn_01x09_Pin, J7 Conn_01x05_Pin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

Commit message: Uodate LQFP64
Routing:
- net TXD: track 28.3 -> 27.7 mm
Changed lines of the file:
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@@
   (segment (start 163.9 73.8) (end 159.7 73.8) (width 0.5) (layer "F.Cu") (net 9))
   (segment (start 155.05 71.75) (end 156.3 73) (width 0.3) (layer "F.Cu") (net 9))
-  (segment (start 144.5 67.3) (end 143.175 68.625) (width 0.5) (layer "F.Cu") (net 10))
-  (segment (start 153.72 65.1) (end 153.72 63.72) (width 0.5) (layer "F.Cu") (net 10))
-  (segment (start 146.8 67.3) (end 144.5 67.3) (width 0.5) (layer "F.Cu") (net 10))
-  (segment (start 149.5 65.5) (end 148.5 66.5) (width 0.5) (layer "F.Cu") (net 10))
-  (segment (start 153.72 63.72) (end 153.2 63.2) (width 0.5) (layer "F.Cu") (net 10))
-  (segment (start 143.175 68.625) (end 143.175 69.5) (width 0.5) (layer "F.Cu") (net 10))
-  (segment (start 148.5 66.5) (end 147.6 66.5) (width 0.5) (layer "F.Cu") (net 10))
+  (segment (start 149.5 64.6) (end 150.9 63.2) (width 0.5) (layer "F.Cu") (net 10))
+  (segment (start 147.8 64.6) (end 149.5 64.6) (width 0.5) (layer "F.Cu") (net 10))
+  (segment (start 143.175 68.625) (end 144.5 67.3) (width 0.5) (layer "F.Cu") (net 10))
   (segment (start 141.35 73.25) (end 142.7 74.6) (width 0.3) (layer "F.Cu") (net 10))
+  (segment (start 144.5 67.3) (end 145.1 67.3) (width 0.5) (layer "F.Cu") (net 10))
   (segment (start 136.075 73.25) (end 141.35 73.25) (width 0.3) (layer "F.Cu") (net 10))
-  (segment (start 149.5 64.6) (end 149.5 65.5) (width 0.5) (layer "F.Cu") (net 10))
-  (segment (start 153.2 63.2) (end 150.9 63.2) (width 0.5) (layer "F.Cu") (net 10))
-  (segment (start 147.6 66.5) (end 146.8 67.3) (width 0.5) (layer "F.Cu") (net 10))
-  (segment (start 150.9 63.2) (end 149.5 64.6) (width 0.5) (layer "F.Cu") (net 10))
+  (segment (start 153.72 63.72) (end 153.72 65.1) (width 0.5) (layer "F.Cu") (net 10))
+  (segment (start 145.1 67.3) (end 147.8 64.6) (width 0.5) (layer "F.Cu") (net 10))
+  (segment (start 153.2 63.2) (end 153.72 63.72) (width 0.5) (layer "F.Cu") (net 10))
+  (segment (start 143.175 69.5) (end 143.175 68.625) (width 0.5) (layer "F.Cu") (net 10))
+  (segment (start 150.9 63.2) (end 153.2 63.2) (width 0.5) (layer "F.Cu") (net 10))
   (via (at 142.7 74.6) (size 0.8) (drill 0.4) (layers "F.Cu" "B.Cu") (net 10))
   (segment (start 143.175 74.125) (end 142.7 74.6) (width 0.5) (layer "B.Cu") (net 10))
