File: circuit/kicad/custom_esp12f/custom_esp12f.kicad_sch (KiCad schematic)
At the start: 17 parts, among them J1 USB_B, SW1 SW_Push, SW2 SW_Push, U1 CH340C, U2 ESP-12F, U3 AMS1117-3.3

Commit message: ESP-12F
Other:
- title: Minimal ESP12-F Module -> Minimal ESP-12F Module
Changed lines of the file:
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@@
   (paper "A5")
   (title_block
-    (title "Minimal ESP12-F Module")
+    (title "Minimal ESP-12F Module")
     (date "2023-10-09")
     (rev "v0")
