File: embedded/esp32/sndin/circuit/sndin.kicad_sch (KiCad schematic)
At the start: 4 parts, among them J1 SPH0645, U1 ESP32-WROOM-32

Commit message: SPH0645 All Zero
Connections:
- net GND: now also J1.1 (Pin_1); no longer J1.2 (Pin_2)
- net MIC_BCLK: now also U1.13 (IO14); no longer U1.30 (IO18)
- net MIC_DATA: now also U1.37 (IO23); no longer U1.31 (IO19)
- net MIC_LRC: now reaches U1.23 (IO15)
- net MIC_LRC: now also J1.2 (Pin_2)
- net MIC_SEL: no longer names the net of U1.29 (IO5)
- net MIC_SEL: no longer J1.1 (Pin_1)
Other:
- moved on the sheet: J1
Changed lines of the file:
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@@
   (no_connect (at 71.12 68.58))
   (no_connect (at 71.12 81.28))
+  (no_connect (at 71.12 55.88))
+  (no_connect (at 71.12 73.66))
+  (no_connect (at 71.12 76.2))
   (no_connect (at 71.12 60.96))
   (no_connect (at 40.64 50.8))
@@
   (no_connect (at 71.12 88.9))
   (no_connect (at 40.64 76.2))
-  (no_connect (at 71.12 83.82))
   (no_connect (at 71.12 93.98))
   (no_connect (at 40.64 81.28))
   (no_connect (at 71.12 43.18))
-  (no_connect (at 71.12 66.04))
   (no_connect (at 71.12 58.42))
   (no_connect (at 71.12 101.6))
@@
   (no_connect (at 71.12 99.06))
   (no_connect (at 71.12 53.34))
-  (no_connect (at 71.12 63.5))
   (no_connect (at 40.64 86.36))
   (no_connect (at 40.64 73.66))
   (no_connect (at 71.12 71.12))
   (no_connect (at 71.12 86.36))
-  (wire (pts (xy 91.44 74.93) (xy 106.68 74.93))
+  (wire (pts (xy 85.09 76.2) (xy 100.33 76.2))
     (stroke (width 0) (type default))
   )
@@
     (stroke (width 0) (type default))
   )
-  (text_box "Mic Pinout:\n\nSEL -> D5\nLRC -> GND\nDATA -> D19\nBCLK -> D18\nGND -> GND\n3V -> VDD\n"
-    (at 124.46 60.96 0) (size 19.05 19.05)
+  (text_box "Mic Pinout:\n\nSEL -> GND\nLRC -> IO15\nDATA -> IO23\nBCLK -> IO14\nGND -> GND\n3V -> VDD\n"
+    (at 110.49 66.04 0) (size 19.05 19.05)
     (stroke (width 0) (type default))
     (fill (type none))
     (effects (font (size 1.27 1.27)) (justify left top))
   )
-  (global_label "MIC_BCLK" (shape input) (at 106.68 69.85 180) (fields_autoplaced)
+  (global_label "MIC_BCLK" (shape input) (at 100.33 71.12 180) (fields_autoplaced)
     (effects (font (size 1.27 1.27)) (justify right))
-    (property "Intersheetrefs" "${INTERSHEET_REFS}" (at 94.5629 69.85 0)
+    (property "Intersheetrefs" "${INTERSHEET_REFS}" (at 88.2129 71.12 0)
       (effects (font (size 1.27 1.27)) (justify right) hide)
     )
   )
-  (global_label "MIC_SEL" (shape input) (at 71.12 55.88 0) (fields_autoplaced)
-    (effects (font (size 1.27 1.27)) (justify left))
-    (property "Intersheetrefs" "${INTERSHEET_REFS}" (at 81.7856 55.88 0)
-      (effects (font (size 1.27 1.27)) (justify left) hide)
-    )
-  )
-  (global_label "MIC_BCLK" (shape input) (at 71.12 73.66 0) (fields_autoplaced)
-    (effects (font (size 1.27 1.27)) (justify left))
-    (property "Intersheetrefs" "${INTERSHEET_REFS}" (at 83.2371 73.66 0)
+  (global_label "MIC_SEL" (shape input) (at 95.25 80.01 0) (fields_autoplaced)
+    (effects (font (size 1.27 1.27)) (justify left))
+    (property "Intersheetrefs" "${INTERSHEET_REFS}" (at 105.9156 80.01 0)
+      (effects (font (size 1.27 1.27)) (justify left) hide)
+    )
+  )
+  (global_label "MIC_BCLK" (shape input) (at 71.12 63.5 0) (fields_autoplaced)
+    (effects (font (size 1.27 1.27)) (justify left))
+    (property "Intersheetrefs" "${INTERSHEET_REFS}" (at 83.2371 63.5 0)
       (effects (font (size 1.27 1.27)) (justify left) hide)
     )
@@
     )
   )
-  (global_label "MIC_DATA" (shape input) (at 106.68 67.31 180) (fields_autoplaced)
+  (global_label "MIC_DATA" (shape input) (at 100.33 68.58 180) (fields_autoplaced)
     (effects (font (size 1.27 1.27)) (justify right))
-    (property "Intersheetrefs" "${INTERSHEET_REFS}" (at 94.9862 67.31 0)
+    (property "Intersheetrefs" "${INTERSHEET_REFS}" (at 88.6362 68.58 0)
       (effects (font (size 1.27 1.27)) (justify right) hide)
     )
@@
     )
   )
-  (global_label "MIC_SEL" (shape input) (at 106.68 62.23 180) (fields_autoplaced)
+  (global_label "MIC_SEL" (shape input) (at 100.33 63.5 180) (fields_autoplaced)
     (effects (font (size 1.27 1.27)) (justify right))
-    (property "Intersheetrefs" "${INTERSHEET_REFS}" (at 96.0144 62.23 0)
+    (property "Intersheetrefs" "${INTERSHEET_REFS}" (at 89.6644 63.5 0)
       (effects (font (size 1.27 1.27)) (justify right) hide)
     )
   )
-  (global_label "MIC_LRC" (shape input) (at 106.68 64.77 180) (fields_autoplaced)
+  (global_label "MIC_LRC" (shape input) (at 100.33 66.04 180) (fields_autoplaced)
     (effects (font (size 1.27 1.27)) (justify right))
-    (property "Intersheetrefs" "${INTERSHEET_REFS}" (at 95.8329 64.77 0)
+    (property "Intersheetrefs" "${INTERSHEET_REFS}" (at 89.4829 66.04 0)
       (effects (font (size 1.27 1.27)) (justify right) hide)
     )
   )
-  (global_label "MIC_LRC" (shape input) (at 101.6 78.74 0) (fields_autoplaced)
-    (effects (font (size 1.27 1.27)) (justify left))
-    (property "Intersheetrefs" "${INTERSHEET_REFS}" (at 112.4471 78.74 0)
-      (effects (font (size 1.27 1.27)) (justify left) hide)
-    )
-  )
-  (global_label "MIC_DATA" (shape input) (at 71.12 76.2 0) (fields_autoplaced)
-    (effects (font (size 1.27 1.27)) (justify left))
-    (property "Intersheetrefs" "${INTERSHEET_REFS}" (at 82.8138 76.2 0)
+  (global_label "MIC_LRC" (shape input) (at 71.12 66.04 0) (fields_autoplaced)
+    (effects (font (size 1.27 1.27)) (justify left))
+    (property "Intersheetrefs" "${INTERSHEET_REFS}" (at 81.9671 66.04 0)
+      (effects (font (size 1.27 1.27)) (justify left) hide)
+    )
+  )
+  (global_label "MIC_DATA" (shape input) (at 71.12 83.82 0) (fields_autoplaced)
+    (effects (font (size 1.27 1.27)) (justify left))
+    (property "Intersheetrefs" "${INTERSHEET_REFS}" (at 82.8138 83.82 0)
       (effects (font (size 1.27 1.27)) (justify left) hide)
     )
@@
     )
   )
-  (symbol (lib_id "Connector:Conn_01x06_Socket") (at 111.76 67.31 0) (unit 1)
-    (in_bom yes) (on_board yes) (dnp no) (fields_autoplaced)
-    (property "Reference" "J1" (at 113.03 67.31 0)
-      (effects (font (size 1.27 1.27)) (justify left))
-    )
-    (property "Value" "SPH0645" (at 113.03 69.85 0)
-      (effects (font (size 1.27 1.27)) (justify left))
-    )
-    (property "Footprint" "" (at 111.76 67.31 0)
-      (effects (font (size 1.27 1.27)) hide)
-    )
-    (property "Datasheet" "~" (at 111.76 67.31 0)
+  (symbol (lib_id "Connector:Conn_01x06_Socket") (at 105.41 68.58 0) (unit 1)
+    (in_bom yes) (on_board yes) (dnp no)
+    (property "Reference" "J1" (at 106.68 63.5 0)
+      (effects (font (size 1.27 1.27)) (justify left))
+    )
+    (property "Value" "SPH0645" (at 99.06 59.69 0)
+      (effects (font (size 1.27 1.27)) (justify left))
+    )
+    (property "Footprint" "" (at 105.41 68.58 0)
+      (effects (font (size 1.27 1.27)) hide)
+    )
+    (property "Datasheet" "~" (at 105.41 68.58 0)
       (effects (font (size 1.27 1.27)) hide)
     )
@@
     )
   )
-  (symbol (lib_id "power:GND") (at 106.68 72.39 270) (unit 1)
-    (in_bom yes) (on_board yes) (dnp no) (fields_autoplaced)
-    (property "Reference" "#PWR02" (at 100.33 72.39 0)
-      (effects (font (size 1.27 1.27)) hide)
-    )
-    (property "Value" "GND" (at 101.6 72.39 0)
-      (effects (font (size 1.27 1.27)) hide)
-    )
-    (property "Footprint" "" (at 106.68 72.39 0)
-      (effects (font (size 1.27 1.27)) hide)
-    )
-    (property "Datasheet" "" (at 106.68 72.39 0)
+  (symbol (lib_id "power:GND") (at 100.33 73.66 270) (unit 1)
+    (in_bom yes) (on_board yes) (dnp no) (fields_autoplaced)
+    (property "Reference" "#PWR02" (at 93.98 73.66 0)
+      (effects (font (size 1.27 1.27)) hide)
+    )
+    (property "Value" "GND" (at 95.25 73.66 0)
+      (effects (font (size 1.27 1.27)) hide)
+    )
+    (property "Footprint" "" (at 100.33 73.66 0)
+      (effects (font (size 1.27 1.27)) hide)
+    )
+    (property "Datasheet" "" (at 100.33 73.66 0)
       (effects (font (size 1.27 1.27)) hide)
     )
@@
     )
   )
-  (symbol (lib_id "power:VDD") (at 91.44 74.93 0) (unit 1)
-    (in_bom yes) (on_board yes) (dnp no) (fields_autoplaced)
-    (property "Reference" "#PWR01" (at 91.44 78.74 0)
-      (effects (font (size 1.27 1.27)) hide)
-    )
-    (property "Value" "VDD" (at 91.44 69.85 0)
+  (symbol (lib_id "power:VDD") (at 85.09 76.2 0) (unit 1)
+    (in_bom yes) (on_board yes) (dnp no) (fields_autoplaced)
+    (property "Reference" "#PWR01" (at 85.09 80.01 0)
+      (effects (font (size 1.27 1.27)) hide)
+    )
+    (property "Value" "VDD" (at 85.09 71.12 0)
       (effects (font (size 1.27 1.27)))
     )
-    (property "Footprint" "" (at 91.44 74.93 0)
-      (effects (font (size 1.27 1.27)) hide)
-    )
-    (property "Datasheet" "" (at 91.44 74.93 0)
+    (property "Footprint" "" (at 85.09 76.2 0)
+      (effects (font (size 1.27 1.27)) hide)
+    )
+    (property "Datasheet" "" (at 85.09 76.2 0)
       (effects (font (size 1.27 1.27)) hide)
     )
@@
     )
   )
-  (symbol (lib_id "power:GND") (at 101.6 78.74 270) (unit 1)
-    (in_bom yes) (on_board yes) (dnp no) (fields_autoplaced)
-    (property "Reference" "#PWR07" (at 95.25 78.74 0)
-      (effects (font (size 1.27 1.27)) hide)
-    )
-    (property "Value" "GND" (at 96.52 78.74 0)
-      (effects (font (size 1.27 1.27)) hide)
-    )
-    (property "Footprint" "" (at 101.6 78.74 0)
-      (effects (font (size 1.27 1.27)) hide)
-    )
-    (property "Datasheet" "" (at 101.6 78.74 0)
-      (effects (font (size 1.27 1.27)) hide)
-    )
+  (symbol (lib_id "power:GND") (at 95.25 80.01 270) (unit 1)
+    (in_bom yes) (on_board yes) (dnp no) (fields_autoplaced)
+    (property "Reference" "#PWR07" (at 88.9 80.01 0)
+      (effects (font (size 1.27 1.27)) hide)
+    )
+    (property "Value" "GND" (at 90.17 80.01 0)
+      (effects (font (size 1.27 1.27)) hide)
+    )
+    (property "Footprint" "" (at 95.25 80.01 0)
+      (effects (font (size 1.27 1.27)) hide)
+    )
+    (property "Datasheet" "" (at 95.25 80.01 0)
+      (effects (font (size 1.27 1.27)) hide)
+    )
